Commit message: new update with downgrade sim from ubuntu 24.04 ros2 jazzy gazebo harmony to ubuntu 22.04 ros2 humble gazebo ignition 6

File: src/gazebo_ackermann_steering_vehicle/model/vehicle.xacro (robot description, xacro)
@@ -190,5 +190,5 @@
     </collision>
     <inertial>
-      <mass value="2"/>
+      <mass value="${wheel_mass}"/>
       <inertia ixx="${wheel_inertia_x}" ixy="0.0" ixz="0.0" iyy="${wheel_inertia_y}" iyz="0" izz="${wheel_inertia_z}"/>
       <origin xyz="0.0 0.0 0.0" rpy="1.570795 0.0 0.0"/>
@@ -213,5 +213,5 @@
     </collision>
     <inertial>
-      <mass value="2"/>
+      <mass value="${wheel_mass}"/>
       <inertia ixx="${wheel_inertia_x}" ixy="0.0" ixz="0.0" iyy="${wheel_inertia_y}" iyz="0" izz="${wheel_inertia_z}"/>
       <origin xyz="0.0 0.0 0.0" rpy="1.570795 0.0 0.0"/>
@@ -280,5 +280,5 @@
     <axis xyz="0 0 1"/>
     <limit effort="${max_steering_effort}" lower="${-max_steering_angle}" upper="${max_steering_angle}" velocity="${max_steering_angular_velocity}"/>
-    <dynamics damping="0.1" friction="0.1"/>
+    <dynamics damping="0.01" friction="0.01"/>
   </joint>
   <!-- Front Left Wheel Joint -->
@@ -289,5 +289,5 @@
     <axis xyz="0 1 0"/>
     <limit effort="${max_effort}" velocity="${max_wheel_angular_velocity}"/>
-    <dynamics damping="0.1" friction="0.1"/>
+    <dynamics damping="0.001" friction="0.0"/>
   </joint>
   <!-- Front Right Steering Joint -->
@@ -298,5 +298,5 @@
     <axis xyz="0 0 1"/>
     <limit effort="${max_steering_effort}" lower="${-max_steering_angle}" upper="${max_steering_angle}" velocity="${max_steering_angular_velocity}"/>
-    <dynamics damping="0.1" friction="0.1"/>
+    <dynamics damping="0.01" friction="0.01"/>
   </joint>
   <!-- Front Right Wheel Joint -->
@@ -307,5 +307,5 @@
     <axis xyz="0 1 0"/>
     <limit effort="${max_effort}" velocity="${max_wheel_angular_velocity}"/>
-    <dynamics damping="0.1" friction="0.1"/>
+    <dynamics damping="0.001" friction="0.0"/>
   </joint>
   <!-- Rear Left Wheel Joint -->
@@ -316,5 +316,5 @@
     <axis xyz="0 1 0"/>
     <limit effort="${max_effort}" velocity="${max_wheel_angular_velocity}"/>
-    <dynamics damping="0.1" friction="0.1"/>
+    <dynamics damping="0.001" friction="0.0"/>
   </joint>
   <!-- Rear Right Wheel Joint -->
@@ -325,5 +325,5 @@
     <axis xyz="0 1 0"/>
     <limit effort="${max_effort}" velocity="${max_wheel_angular_velocity}"/>
-    <dynamics damping="0.1" friction="0.1"/>
+    <dynamics damping="0.001" friction="0.0"/>
   </joint>
   <!-- IMU Joint -->
